File: microphone.sch (KiCad schematic (older format))
At the start: 24 parts, among them U2 LM324, U3 MCP73832T-2ACI_OT, U4 LTC2941IMS8EPBF

Commit message: Slight Placement Changes
Other:
- moved on the sheet: C?, D?, J?, R?

Commit message: Motor Controller Done
Parts:
- removed MK?: Microphone_Condenser, symbol Device:Microphone_Condenser
- added C?: 100 uF, symbol Device:CP1_Small
- added C? (x3): 0.1 uF, symbol Device:C_Small
- added C?: 10 nF, symbol Device:C_Small
- added C?: 0.47 uF, symbol Device:C_Small
- added R? (x2): 4.7 k, Resistor_SMD:R_0805_2012Metric_Pad1.15x1.40mm_HandSolder, symbol Device:R_Small_US
- added R?: 1 M, Resistor_SMD:R_0805_2012Metric_Pad1.15x1.40mm_HandSolder, symbol Device:R_Small_US
- added R? (x2): 100 m, Resistor_SMD:R_0805_2012Metric_Pad1.15x1.40mm_HandSolder, symbol Device:R_Small_US
- added R? (x5): 10 k, Resistor_SMD:R_0805_2012Metric_Pad1.15x1.40mm_HandSolder, symbol Device:R_Small_US
- added R?: 1.5 k, Resistor_SMD:R_0805_2012Metric_Pad1.15x1.40mm_HandSolder, symbol Device:R_Small_US
- added RV?: 10k, symbol Device:R_POT_US
- added U?: DRV8825PWP, Texas_Instruments-DRV8825PWP-*, symbol DRV8825PWP:DRV8825PWP
- J?: symbol Connector_Generic:Conn_01x05 -> Connector_Generic:Conn_01x06
- U4: symbol LTC2941IMS8E:LTC2941IMS8EPBF -> noFretTuner-rescue:LTC2941IMS8EPBF-LTC2941IMS8E
Connections:
- net labels added: A1, A2, B1, B2, MOTOR_DECAY, MOTOR_DIR, MOTOR_STEP, MOTOR_nRESET, motor_MODE0, motor_MODE1, motor_MODE2, motor_nENBL, motor_nFAULT, motor_nSLEEP, nHOME
- wire segments 80 -> 164
Other:
- note added: "EN\nVIN\nVIN\nGND\nGND\nVOUT\n"
- note added: "VOUT\nGND\nVIN\nEN\nPG"
- moved on the sheet: C?, D?, J?, R1, R2, R3, R4, R5, R6, R7, R8, R?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

Commit message: First Draft Complete
Parts:
- removed C?: 100 uF, symbol Device:CP1_Small
- removed C? (x3): 0.1 uF, symbol Device:C_Small
- removed C?: 10 nF, symbol Device:C_Small
- removed C?: 0.47 uF, symbol Device:C_Small
- removed R?: 1 M, Resistor_SMD:R_0805_2012Metric_Pad1.15x1.40mm_HandSolder, symbol Device:R_Small_US
- removed R? (x2): 100 m, Resistor_SMD:R_0805_2012Metric_Pad1.15x1.40mm_HandSolder, symbol Device:R_Small_US
- removed R? (x5): 10 k, Resistor_SMD:R_0805_2012Metric_Pad1.15x1.40mm_HandSolder, symbol Device:R_Small_US
- removed R?: 1.5 k, Resistor_SMD:R_0805_2012Metric_Pad1.15x1.40mm_HandSolder, symbol Device:R_Small_US
- removed RV?: 10k, symbol Device:R_POT_US
- removed U?: DRV8825PWP, Texas_Instruments-DRV8825PWP-*, symbol DRV8825PWP:DRV8825PWP
- added C? (x2): ?, symbol Device:C_Small
Connections:
- net labels removed: A1, A2, B1, B2, MOTOR_DECAY, MOTOR_DIR, MOTOR_STEP, MOTOR_nRESET, motor_MODE0, motor_MODE1, motor_MODE2, motor_nENBL, motor_nFAULT, motor_nSLEEP, nHOME
- wire segments 164 -> 96
Other:
- note added: "Battery Charger & Monitor"
- note added: "Microphone Analog Filters"
- moved on the sheet: C?, D?, J?, R1, R2, R3, R4, R5, R6, R7, R8, R?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

Commit message: Ready for PCB Layout
Parts:
- removed C?: 0.1 uF, symbol Device:C_Small
- removed C?: 2.2 uF, symbol Device:C_Small
- removed C? (x2): ?, symbol Device:C_Small
- removed R4, R5: 100, Resistor_SMD:R_0805_2012Metric_Pad1.15x1.40mm_HandSolder, symbol Device:R_Small_US
- removed R6, R7: 1k, Resistor_SMD:R_0805_2012Metric_Pad1.15x1.40mm_HandSolder, symbol Device:R_Small_US
- removed R8: 330, Resistor_SMD:R_0805_2012Metric_Pad1.15x1.40mm_HandSolder, symbol Device:R_Small_US
- removed RV1: 10k, symbol Device:R_POT_US
- removed unit 1 of U2
- removed unit 2 of U2
- added C24, C27: 0.1 uF, symbol Device:C_Small
- added C28: 1 uF, symbol Device:C_Small
- added R27: 1 k, Resistor_SMD:R_0805_2012Metric_Pad1.15x1.40mm_HandSolder, symbol Device:R_Small_US
- added R33: 200, Resistor_SMD:R_0805_2012Metric_Pad1.15x1.40mm_HandSolder, symbol Device:R_Small_US
- added RV2: 1 M, symbol Device:R_POT_US
- added unit 1 of U3
- J10: renamed from J?; footprint (none) -> Connector_PinHeader_2.54mm:PinHeader_1x06_P2.54mm_Vertical
- J9: renamed from J?; footprint (none) -> Connector_PinHeader_2.54mm:PinHeader_1x05_P2.54mm_Vertical
- R26: renamed from R1; value 3.6 k -> 10 k
- R31: renamed from R?; value 100 m -> 25 m
- gave numbers to parts that had none: 8
- renumbered R2 to R28, R3 to R29, U2 to U3, U3 to U5
Connections:
- net labels added: +3.3VA, GNDA
- net labels removed: +3V3
- wire segments 96 -> 90
Other:
- note added: "Low Pass 800 Hz"
- note removed: "Bandpass\n(65.8 hz to 1196 hz)"
- moved on the sheet: C26, R26, R28, R29, U3C, U3E
